Commit message: Changes from hackathon

File: cob_hardware_config/cob3-1/urdf/cob3-1.urdf.xacro (robot description, xacro)
@@ -64,4 +64,24 @@
     </plugin>
   </gazebo>
+  <joint name="$base_extra_collision_joint" type="fixed">
+    <origin xyz="${arm_x - 0.05} ${torso_y} ${arm_z - 0.1}" rpy="0 0 0" />
+    <parent link="base_link"/>
+    <child link="base_extra_collision_link" />
+  </joint>
+  <link name="base_extra_collision_link">
+    <visual>
+      <origin xyz="0 0 0" rpy="0 0 0" />
+      <geometry>
+        <box size="0.20 0.45 0.05"/>
+      </geometry>
+      <material name="IPA/LightGrey"/>
+    </visual>
+    <collision>
+      <origin xyz="0 0 0" rpy="0 0 0" />
+      <geometry>
+        <box size="0.20 0.45 0.05"/>
+      </geometry>
+    </collision>
+  </link>
   <xacro:schunk_sdh name="sdh" parent="arm_7_link">
     <origin xyz="${sdh_x} ${sdh_y} ${sdh_z}" rpy="${sdh_roll} ${sdh_pitch} ${sdh_yaw}" />

Commit message: [Manipulation] make collision box smaller

File: cob_hardware_config/cob3-1/urdf/cob3-1.urdf.xacro (robot description, xacro)
@@ -73,5 +73,5 @@
       <origin xyz="0 0 0" rpy="0 0 0" />
       <geometry>
-        <box size="0.20 0.45 0.05"/>
+        <box size="0.12 0.45 0.05"/>
       </geometry>
       <material name="IPA/LightGrey"/>

Commit message: [robocup2016] uncommitted changes made during robocup 2016

File: cob_hardware_config/cob3-1/urdf/cob3-1.urdf.xacro (robot description, xacro)
@@ -80,5 +80,5 @@
       <origin xyz="0 0 0" rpy="0 0 0" />
       <geometry>
-        <box size="0.20 0.45 0.05"/>
+        <box size="0.12 0.45 0.05"/>
       </geometry>
     </collision>
